Commit message: Add feed forward controller in torque

File: src/allegro_hand_description/allegro_hand_description_left.urdf (robot description, URDF)
Before this commit: robot allegro_hand_left, 21 links, 20 joints
Joints:
- removed joint joint_0.0
- removed joint joint_1.0
- removed joint joint_10.0
- removed joint joint_11.0
- removed joint joint_11.0_tip
- removed joint joint_12.0
- removed joint joint_13.0
- removed joint joint_14.0
- removed joint joint_15.0
- removed joint joint_15.0_tip
- removed joint joint_2.0
- removed joint joint_3.0
- removed joint joint_3.0_tip
- removed joint joint_4.0
- removed joint joint_5.0
- removed joint joint_6.0
- removed joint joint_7.0
- removed joint joint_7.0_tip
- removed joint joint_8.0
- removed joint joint_9.0
- added joint joint_0: type revolute, parent palm_link, child link_0.0, origin xyz=0 -0.0435 -0.001542 rpy=0.08726646255 0 0, axis 0 0 1, limit lower=-0.47 upper=0.47 effort=15 velocity=7
- added joint joint_1: type revolute, parent link_0.0, child link_1.0, origin xyz=0 0 0.0164, axis 0 1 0, limit lower=-0.196 upper=1.61 effort=15 velocity=7
- added joint joint_10: type revolute, parent link_9.0, child link_10.0, origin xyz=0 0 0.054, axis 0 1 0, limit lower=-0.174 upper=1.709 effort=15 velocity=7
- added joint joint_11: type revolute, parent link_10.0, child link_11.0, origin xyz=0 0 0.0384, axis 0 1 0, limit lower=-0.227 upper=1.618 effort=15 velocity=7
- added joint joint_11_tip: type fixed, parent link_11.0, child link_11.0_tip, origin xyz=0 0 0.0267 rpy=0 0 0
- added joint joint_12: type revolute, parent palm_link, child link_12.0, origin xyz=-0.0182 -0.019333 -0.045987 rpy=0 -1.65806278845 1.5707963259, axis +1 0 0, limit lower=0.263 upper=1.396 effort=15 velocity=7
- added joint joint_13: type revolute, parent link_12.0, child link_13.0, origin xyz=-0.027 -0.005 0.0399, axis 0 0 -1, limit lower=-0.105 upper=1.163 effort=15 velocity=7
- added joint joint_14: type revolute, parent link_13.0, child link_14.0, origin xyz=0 0 0.0177, axis 0 1 0, limit lower=-0.189 upper=1.644 effort=15 velocity=7
- added joint joint_15: type revolute, parent link_14.0, child link_15.0, origin xyz=0 0 0.0514, axis 0 1 0, limit lower=-0.162 upper=1.719 effort=15 velocity=7
- added joint joint_15_tip: type fixed, parent link_15.0, child link_15.0_tip, origin xyz=0 0 0.0423 rpy=0 0 0
- added joint joint_2: type revolute, parent link_1.0, child link_2.0, origin xyz=0 0 0.054, axis 0 1 0, limit lower=-0.174 upper=1.709 effort=15 velocity=7
- added joint joint_3: type revolute, parent link_2.0, child link_3.0, origin xyz=0 0 0.0384, axis 0 1 0, limit lower=-0.227 upper=1.618 effort=15 velocity=7
- added joint joint_3_tip: type fixed, parent link_3.0, child link_3.0_tip, origin xyz=0 0 0.0267 rpy=0 0 0
- added joint joint_4: type revolute, parent palm_link, child link_4.0, origin xyz=0 0 0.0007 rpy=0.0 0 0, axis 0 0 1, limit lower=-0.47 upper=0.47 effort=15 velocity=7
- added joint joint_5: type revolute, parent link_4.0, child link_5.0, origin xyz=0 0 0.0164, axis 0 1 0, limit lower=-0.196 upper=1.61 effort=15 velocity=7
- added joint joint_6: type revolute, parent link_5.0, child link_6.0, origin xyz=0 0 0.054, axis 0 1 0, limit lower=-0.174 upper=1.709 effort=15 velocity=7
- added joint joint_7: type revolute, parent link_6.0, child link_7.0, origin xyz=0 0 0.0384, axis 0 1 0, limit lower=-0.227 upper=1.618 effort=15 velocity=7
- added joint joint_7_tip: type fixed, parent link_7.0, child link_7.0_tip, origin xyz=0 0 0.0267 rpy=0 0 0
- added joint joint_8: type revolute, parent palm_link, child link_8.0, origin xyz=0 0.0435 -0.001542 rpy=-0.08726646255 0 0, axis 0 0 1, limit lower=-0.47 upper=0.47 effort=15 velocity=7
- added joint joint_9: type revolute, parent link_8.0, child link_9.0, origin xyz=0 0 0.0164, axis 0 1 0, limit lower=-0.196 upper=1.61 effort=15 velocity=7

File: src/allegro_hand_description/allegro_hand_description_right.urdf (robot description, URDF)
Before this commit: robot allegro_hand_right, 21 links, 20 joints
Joints:
- removed joint joint_0.0
- removed joint joint_1.0
- removed joint joint_10.0
- removed joint joint_11.0
- removed joint joint_11.0_tip
- removed joint joint_12.0
- removed joint joint_13.0
- removed joint joint_14.0
- removed joint joint_15.0
- removed joint joint_15.0_tip
- removed joint joint_2.0
- removed joint joint_3.0
- removed joint joint_3.0_tip
- removed joint joint_4.0
- removed joint joint_5.0
- removed joint joint_6.0
- removed joint joint_7.0
- removed joint joint_7.0_tip
- removed joint joint_8.0
- removed joint joint_9.0
- added joint joint_0: type revolute, parent palm_link, child link_0.0, origin xyz=0 0.0435 -0.001542 rpy=-0.08726646255 0 0, axis 0 0 1, limit lower=-0.47 upper=0.47 effort=15 velocity=7
- added joint joint_1: type revolute, parent link_0.0, child link_1.0, origin xyz=0 0 0.0164, axis 0 1 0, limit lower=-0.196 upper=1.61 effort=15 velocity=7
- added joint joint_10: type revolute, parent link_9.0, child link_10.0, origin xyz=0 0 0.054, axis 0 1 0, limit lower=-0.174 upper=1.709 effort=15 velocity=7
- added joint joint_11: type revolute, parent link_10.0, child link_11.0, origin xyz=0 0 0.0384, axis 0 1 0, limit lower=-0.227 upper=1.618 effort=15 velocity=7
- added joint joint_11_tip: type fixed, parent link_11.0, child link_11.0_tip, origin xyz=0 0 0.0267 rpy=0 0 0
- added joint joint_12: type revolute, parent palm_link, child link_12.0, origin xyz=-0.0182 0.019333 -0.045987 rpy=0 -1.65806278845 -1.5707963259, axis -1 0 0, limit lower=0.263 upper=1.396 effort=15 velocity=7
- added joint joint_13: type revolute, parent link_12.0, child link_13.0, origin xyz=-0.027 0.005 0.0399, axis 0 0 1, limit lower=-0.105 upper=1.163 effort=15 velocity=7
- added joint joint_14: type revolute, parent link_13.0, child link_14.0, origin xyz=0 0 0.0177, axis 0 1 0, limit lower=-0.189 upper=1.644 effort=15 velocity=7
- added joint joint_15: type revolute, parent link_14.0, child link_15.0, origin xyz=0 0 0.0514, axis 0 1 0, limit lower=-0.162 upper=1.719 effort=15 velocity=7
- added joint joint_15_tip: type fixed, parent link_15.0, child link_15.0_tip, origin xyz=0 0 0.0423 rpy=0 0 0
- added joint joint_2: type revolute, parent link_1.0, child link_2.0, origin xyz=0 0 0.054, axis 0 1 0, limit lower=-0.174 upper=1.709 effort=15 velocity=7
- added joint joint_3: type revolute, parent link_2.0, child link_3.0, origin xyz=0 0 0.0384, axis 0 1 0, limit lower=-0.227 upper=1.618 effort=15 velocity=7
- added joint joint_3_tip: type fixed, parent link_3.0, child link_3.0_tip, origin xyz=0 0 0.0267 rpy=0 0 0
- added joint joint_4: type revolute, parent palm_link, child link_4.0, origin xyz=0 0 0.0007 rpy=0.0 0 0, axis 0 0 1, limit lower=-0.47 upper=0.47 effort=15 velocity=7
- added joint joint_5: type revolute, parent link_4.0, child link_5.0, origin xyz=0 0 0.0164, axis 0 1 0, limit lower=-0.196 upper=1.61 effort=15 velocity=7
- added joint joint_6: type revolute, parent link_5.0, child link_6.0, origin xyz=0 0 0.054, axis 0 1 0, limit lower=-0.174 upper=1.709 effort=15 velocity=7
- added joint joint_7: type revolute, parent link_6.0, child link_7.0, origin xyz=0 0 0.0384, axis 0 1 0, limit lower=-0.227 upper=1.618 effort=15 velocity=7
- added joint joint_7_tip: type fixed, parent link_7.0, child link_7.0_tip, origin xyz=0 0 0.0267 rpy=0 0 0
- added joint joint_8: type revolute, parent palm_link, child link_8.0, origin xyz=0 -0.0435 -0.001542 rpy=0.08726646255 0 0, axis 0 0 1, limit lower=-0.47 upper=0.47 effort=15 velocity=7
- added joint joint_9: type revolute, parent link_8.0, child link_9.0, origin xyz=0 0 0.0164, axis 0 1 0, limit lower=-0.196 upper=1.61 effort=15 velocity=7
