Commit message: Fix TF in RVIZ

File: src/allegro_hand_description/allegro_hand_description_right.xacro (robot description, xacro)
@@ -99,5 +99,5 @@
             </inertial>
         </link>
-        <joint name="joint_${finger_num*4+0}.0" type="revolute">
+        <joint name="joint_${finger_num*4+0}" type="revolute">
             <axis xyz="-1 0 0"/>
             <limit effort="15" velocity="7"
@@ -134,5 +134,5 @@
             </inertial>
         </link>
-        <joint name="joint_${finger_num*4+1}.0" type="revolute">
+        <joint name="joint_${finger_num*4+1}" type="revolute">
             <axis xyz="0 0 1"/>
             <limit effort="15" velocity="7"
@@ -166,5 +166,5 @@
             </inertial>
         </link>
-        <joint name="joint_${finger_num*4+2}.0" type="revolute">
+        <joint name="joint_${finger_num*4+2}" type="revolute">
             <axis xyz="0 1 0"/>
             <limit effort="15" velocity="7"
@@ -199,5 +199,5 @@
             </inertial>
         </link>
-        <joint name="joint_${finger_num*4+3}.0" type="revolute">
+        <joint name="joint_${finger_num*4+3}" type="revolute">
             <axis xyz="0 1 0"/>
             <limit effort="15" velocity="7"
@@ -265,5 +265,5 @@
             </inertial>
         </link>
-        <joint name="joint_${finger_num*4+0}.0" type="revolute">
+        <joint name="joint_${finger_num*4+0}" type="revolute">
             <axis xyz="0 0 1"/>
             <limit effort="15" velocity="7"
@@ -298,5 +298,5 @@
             </inertial>
         </link>
-        <joint name="joint_${finger_num*4+1}.0" type="revolute">
+        <joint name="joint_${finger_num*4+1}" type="revolute">
             <limit effort="15" velocity="7"
                    lower="${limit_1_low+joint_safety_margin}"
@@ -330,5 +330,5 @@
             </inertial>
         </link>
-        <joint name="joint_${finger_num*4+2}.0" type="revolute">
+        <joint name="joint_${finger_num*4+2}" type="revolute">
             <axis xyz="0 1 0"/>
             <limit effort="15" velocity="7"
@@ -362,5 +362,5 @@
             </inertial>
         </link>
-        <joint name="joint_${finger_num*4+3}.0" type="revolute">
+        <joint name="joint_${finger_num*4+3}" type="revolute">
             <axis xyz="0 1 0"/>
             <limit effort="15" velocity="7"
