Commit message: Renaming joint alphabetically

File: src/allegro_hand_description/allegro_hand_description.xacro (robot description, xacro)
@@ -85,5 +85,5 @@
                  params="finger_num offset_origin_x offset_origin_y offset_origin_z finger_angle_r finger_angle_p finger_angle_y">
         <!-- [LINK 12] -->
-        <link name="link_${finger_num*4+0}">
+        <link name="link_${'%02d' % (finger_num*4+0)}">
             <visual>
                 <geometry>
@@ -109,5 +109,5 @@
             </inertial>
         </link>
-        <joint name="joint_${finger_num*4+0}" type="revolute">
+        <joint name="joint_${'%02d' % (finger_num*4+0)}" type="revolute">
             <axis xyz="${minus_right} 0 0"/>
             <limit effort="15" velocity="7"
@@ -115,5 +115,5 @@
                    upper="${limit_0_t_up-joint_safety_margin}"/>
             <parent link="palm_link"/>
-            <child link="link_${finger_num*4+0}"/>
+            <child link="link_${'%02d' % (finger_num*4+0)}"/>
             <origin rpy="${finger_angle_r} ${finger_angle_p} ${finger_angle_y}"
                     xyz="${offset_origin_x} ${offset_origin_y} ${offset_origin_z}"/>
@@ -121,5 +121,5 @@
         </joint>
         <!-- [LINK 13] -->
-        <link name="link_${finger_num*4+1}">
+        <link name="link_${'%02d' % (finger_num*4+1)}">
             <visual>
                 <geometry>
@@ -144,16 +144,16 @@
             </inertial>
         </link>
-        <joint name="joint_${finger_num*4+1}" type="revolute">
+        <joint name="joint_${'%02d' % (finger_num*4+1)}" type="revolute">
             <axis xyz="0 0 ${minus_left}"/>
             <limit effort="15" velocity="7"
                    lower="${limit_1_t_low+joint_safety_margin}"
                    upper="${limit_1_t_up-joint_safety_margin}"/>
-            <parent link="link_${finger_num*4+0}"/>
-            <child link="link_${finger_num*4+1}"/>
+            <parent link="link_${'%02d' % (finger_num*4+0)}"/>
+            <child link="link_${'%02d' % (finger_num*4+1)}"/>
             <origin xyz="-0.027 ${minus_left * 0.005} 0.0399"/>
             <dynamics damping="3" friction="5"/>
         </joint>
         <!-- [LINK 14] -->
-        <link name="link_${finger_num*4+2}">
+        <link name="link_${'%02d' % (finger_num*4+2)}">
             <visual>
                 <geometry>
@@ -176,16 +176,16 @@
             </inertial>
         </link>
-        <joint name="joint_${finger_num*4+2}" type="revolute">
+        <joint name="joint_${'%02d' % (finger_num*4+2)}" type="revolute">
             <axis xyz="0 1 0"/>
             <limit effort="15" velocity="7"
                    lower="${limit_2_t_low+joint_safety_margin}"
                    upper="${limit_2_t_up-joint_safety_margin}"/>
-            <parent link="link_${finger_num*4+1}"/>
-            <child link="link_${finger_num*4+2}"/>
+            <parent link="link_${'%02d' % (finger_num*4+1)}"/>
+            <child link="link_${'%02d' % (finger_num*4+2)}"/>
             <origin xyz="0 0 ${link1_t_z}"/>
             <dynamics damping="3" friction="10"/>
         </joint>
         <!-- [LINK 15] -->
-        <link name="link_${finger_num*4+3}">
+        <link name="link_${'%02d' % (finger_num*4+3)}">
             <visual>
                 <geometry>
@@ -209,16 +209,16 @@
             </inertial>
         </link>
-        <joint name="joint_${finger_num*4+3}" type="revolute">
+        <joint name="joint_${'%02d' % (finger_num*4+3)}" type="revolute">
             <axis xyz="0 1 0"/>
             <limit effort="15" velocity="7"
                    lower="${limit_3_t_low+joint_safety_margin}"
                    upper="${limit_3_t_up-joint_safety_margin}"/>
-            <parent link="link_${finger_num*4+2}"/>
-            <child link="link_${finger_num*4+3}"/>
+            <parent link="link_${'%02d' % (finger_num*4+2)}"/>
+            <child link="link_${'%02d' % (finger_num*4+3)}"/>
             <origin xyz="0 0 ${link2_t_z}"/>
             <dynamics damping="3" friction="12"/>
         </joint>
         <!-- [FINGER TIP] -->
-        <link name="link_${finger_num*4+3}_tip">
+        <link name="link_${'%02d' % (finger_num*4+3)}_tip">
             <visual>
                 <geometry>
@@ -243,7 +243,7 @@
             </inertial>
         </link>
-        <joint name="joint_${finger_num*4+3}_tip" type="fixed">
-            <parent link="link_${finger_num*4+3}"/>
-            <child link="link_${finger_num*4+3}_tip"/>
+        <joint name="joint_${'%02d' % (finger_num*4+3)}_tip" type="fixed">
+            <parent link="link_${'%02d' % (finger_num*4+3)}"/>
+            <child link="link_${'%02d' % (finger_num*4+3)}_tip"/>
             <origin rpy="0 0 0" xyz="0 0 ${link3_t_z-fingerTip_r}"/>
         </joint>
@@ -254,5 +254,5 @@
                  params="finger_num offset_origin_x offset_origin_y offset_origin_z finger_angle_r">
         <!-- [LINK 0, 4, 8] -->
-        <link name="link_${finger_num*4+0}">
+        <link name="link_${'%02d' % (finger_num*4+0)}">
             <visual>
                 <geometry>
@@ -275,5 +275,5 @@
             </inertial>
         </link>
-        <joint name="joint_${finger_num*4+0}" type="revolute">
+        <joint name="joint_${'%02d' % (finger_num*4+0)}" type="revolute">
             <axis xyz="0 0 1"/>
             <limit effort="15" velocity="7"
@@ -281,5 +281,5 @@
                    upper="${limit_0_up-joint_safety_margin}"/>
             <parent link="palm_link"/>
-            <child link="link_${finger_num*4+0}"/>
+            <child link="link_${'%02d' % (finger_num*4+0)}"/>
             <origin rpy="${finger_angle_r} 0 0"
                     xyz="${offset_origin_x} ${offset_origin_y} ${offset_origin_z}"/>
@@ -287,5 +287,5 @@
         </joint>
         <!-- [LINK 1, 5, 9] -->
-        <link name="link_${finger_num*4+1}">
+        <link name="link_${'%02d' % (finger_num*4+1)}">
             <visual>
                 <geometry>
@@ -308,16 +308,16 @@
             </inertial>
         </link>
-        <joint name="joint_${finger_num*4+1}" type="revolute">
+        <joint name="joint_${'%02d' % (finger_num*4+1)}" type="revolute">
             <limit effort="15" velocity="7"
                    lower="${limit_1_low+joint_safety_margin}"
                    upper="${limit_1_up-joint_safety_margin}"/>
             <axis xyz="0 1 0"/>
-            <parent link="link_${finger_num*4+0}"/>
-            <child link="link_${finger_num*4+1}"/>
+            <parent link="link_${'%02d' % (finger_num*4+0)}"/>
+            <child link="link_${'%02d' % (finger_num*4+1)}"/>
             <origin xyz="0 0 ${link0_z}"/>
             <dynamics damping="3" friction="5"/>
         </joint>
         <!-- [LINK 2, 6, 10]-->
-        <link name="link_${finger_num*4+2}">
+        <link name="link_${'%02d' % (finger_num*4+2)}">
             <visual>
                 <geometry>
@@ -340,16 +340,16 @@
             </inertial>
         </link>
-        <joint name="joint_${finger_num*4+2}" type="revolute">
+        <joint name="joint_${'%02d' % (finger_num*4+2)}" type="revolute">
             <axis xyz="0 1 0"/>
             <limit effort="15" velocity="7"
                    lower="${limit_2_low+joint_safety_margin}"
                    upper="${limit_2_up-joint_safety_margin}"/>
-            <parent link="link_${finger_num*4+1}"/>
-            <child link="link_${finger_num*4+2}"/>
+            <parent link="link_${'%02d' % (finger_num*4+1)}"/>
+            <child link="link_${'%02d' % (finger_num*4+2)}"/>
             <origin xyz="0 0 ${link1_z}"/>
             <dynamics damping="8" friction="10"/>
         </joint>
         <!-- [LINK 3, 7, 11] -->
-        <link name="link_${finger_num*4+3}">
+        <link name="link_${'%02d' % (finger_num*4+3)}">
             <visual>
                 <geometry>
@@ -372,16 +372,16 @@
             </inertial>
         </link>
-        <joint name="joint_${finger_num*4+3}" type="revolute">
+        <joint name="joint_${'%02d' % (finger_num*4+3)}" type="revolute">
             <axis xyz="0 1 0"/>
             <limit effort="15" velocity="7"
                    lower="${limit_3_low+joint_safety_margin}"
                    upper="${limit_3_up-joint_safety_margin}"/>
-            <parent link="link_${finger_num*4+2}"/>
-            <child link="link_${finger_num*4+3}"/>
+            <parent link="link_${'%02d' % (finger_num*4+2)}"/>
+            <child link="link_${'%02d' % (finger_num*4+3)}"/>
             <origin xyz="0 0 ${link2_z}"/>
             <dynamics damping="10" friction="12"/>
         </joint>
         <!-- [FINGER TIP] -->
-        <link name="link_${finger_num*4+3}_tip">
+        <link name="link_${'%02d' % (finger_num*4+3)}_tip">
             <visual>
                 <geometry>
@@ -405,7 +405,7 @@
             </inertial>
         </link>
-        <joint name="joint_${finger_num*4+3}_tip" type="fixed">
-            <parent link="link_${finger_num*4+3}"/>
-            <child link="link_${finger_num*4+3}_tip"/>
+        <joint name="joint_${'%02d' % (finger_num*4+3)}_tip" type="fixed">
+            <parent link="link_${'%02d' % (finger_num*4+3)}"/>
+            <child link="link_${'%02d' % (finger_num*4+3)}_tip"/>
             <origin rpy="0 0 0" xyz="0 0 ${link3_z-fingerTip_r}"/>
         </joint>

Commit message: More realistic friction value and joint limits

File: src/allegro_hand_description/allegro_hand_description.xacro (robot description, xacro)
@@ -111,6 +111,6 @@
         <joint name="joint_${'%02d' % (finger_num*4+0)}" type="revolute">
             <axis xyz="${minus_right} 0 0"/>
-            <limit effort="15" velocity="7"
-                   lower="${limit_0_t_low-joint_safety_margin}"
+            <limit effort="0.71" velocity="0.12"
+                   lower="${limit_0_t_low+joint_safety_margin}"
                    upper="${limit_0_t_up-joint_safety_margin}"/>
             <parent link="palm_link"/>
@@ -118,5 +118,5 @@
             <origin rpy="${finger_angle_r} ${finger_angle_p} ${finger_angle_y}"
                     xyz="${offset_origin_x} ${offset_origin_y} ${offset_origin_z}"/>
-            <dynamics damping="3" friction="10"/>
+            <dynamics damping="0.01" friction="0.01"/>
         </joint>
         <!-- [LINK 13] -->
@@ -146,5 +146,5 @@
         <joint name="joint_${'%02d' % (finger_num*4+1)}" type="revolute">
             <axis xyz="0 0 ${minus_left}"/>
-            <limit effort="15" velocity="7"
+            <limit effort="0.71" velocity="0.12"
                    lower="${limit_1_t_low+joint_safety_margin}"
                    upper="${limit_1_t_up-joint_safety_margin}"/>
@@ -152,5 +152,5 @@
             <child link="link_${'%02d' % (finger_num*4+1)}"/>
             <origin xyz="-0.027 ${minus_left * 0.005} 0.0399"/>
-            <dynamics damping="3" friction="5"/>
+            <dynamics damping="0.01" friction="0.01"/>
         </joint>
         <!-- [LINK 14] -->
@@ -178,5 +178,5 @@
         <joint name="joint_${'%02d' % (finger_num*4+2)}" type="revolute">
             <axis xyz="0 1 0"/>
-            <limit effort="15" velocity="7"
+            <limit effort="0.71" velocity="0.12"
                    lower="${limit_2_t_low+joint_safety_margin}"
                    upper="${limit_2_t_up-joint_safety_margin}"/>
@@ -184,5 +184,5 @@
             <child link="link_${'%02d' % (finger_num*4+2)}"/>
             <origin xyz="0 0 ${link1_t_z}"/>
-            <dynamics damping="3" friction="10"/>
+            <dynamics damping="0.01" friction="0.01"/>
         </joint>
         <!-- [LINK 15] -->
@@ -211,5 +211,5 @@
         <joint name="joint_${'%02d' % (finger_num*4+3)}" type="revolute">
             <axis xyz="0 1 0"/>
-            <limit effort="15" velocity="7"
+            <limit effort="0.71" velocity="0.12"
                    lower="${limit_3_t_low+joint_safety_margin}"
                    upper="${limit_3_t_up-joint_safety_margin}"/>
@@ -217,5 +217,5 @@
             <child link="link_${'%02d' % (finger_num*4+3)}"/>
             <origin xyz="0 0 ${link2_t_z}"/>
-            <dynamics damping="3" friction="12"/>
+            <dynamics damping="0.01" friction="0.01"/>
         </joint>
         <!-- [FINGER TIP] -->
@@ -277,5 +277,5 @@
         <joint name="joint_${'%02d' % (finger_num*4+0)}" type="revolute">
             <axis xyz="0 0 1"/>
-            <limit effort="15" velocity="7"
+            <limit effort="0.71" velocity="0.12"
                    lower="${limit_0_low+joint_safety_margin}"
                    upper="${limit_0_up-joint_safety_margin}"/>
@@ -284,5 +284,5 @@
             <origin rpy="${finger_angle_r} 0 0"
                     xyz="${offset_origin_x} ${offset_origin_y} ${offset_origin_z}"/>
-            <dynamics damping="3" friction="10"/>
+            <dynamics damping="0.01" friction="0.01"/>
         </joint>
         <!-- [LINK 1, 5, 9] -->
@@ -309,5 +309,5 @@
         </link>
         <joint name="joint_${'%02d' % (finger_num*4+1)}" type="revolute">
-            <limit effort="15" velocity="7"
+            <limit effort="0.71" velocity="0.12"
                    lower="${limit_1_low+joint_safety_margin}"
                    upper="${limit_1_up-joint_safety_margin}"/>
@@ -316,5 +316,5 @@
             <child link="link_${'%02d' % (finger_num*4+1)}"/>
             <origin xyz="0 0 ${link0_z}"/>
-            <dynamics damping="3" friction="5"/>
+            <dynamics damping="0.01" friction="0.01"/>
         </joint>
         <!-- [LINK 2, 6, 10]-->
@@ -342,5 +342,5 @@
         <joint name="joint_${'%02d' % (finger_num*4+2)}" type="revolute">
             <axis xyz="0 1 0"/>
-            <limit effort="15" velocity="7"
+            <limit effort="0.71" velocity="0.12"
                    lower="${limit_2_low+joint_safety_margin}"
                    upper="${limit_2_up-joint_safety_margin}"/>
@@ -348,5 +348,5 @@
             <child link="link_${'%02d' % (finger_num*4+2)}"/>
             <origin xyz="0 0 ${link1_z}"/>
-            <dynamics damping="8" friction="10"/>
+            <dynamics damping="0.01" friction="0.01"/>
         </joint>
         <!-- [LINK 3, 7, 11] -->
@@ -374,5 +374,5 @@
         <joint name="joint_${'%02d' % (finger_num*4+3)}" type="revolute">
             <axis xyz="0 1 0"/>
-            <limit effort="15" velocity="7"
+            <limit effort="0.71" velocity="0.12"
                    lower="${limit_3_low+joint_safety_margin}"
                    upper="${limit_3_up-joint_safety_margin}"/>
@@ -380,5 +380,5 @@
             <child link="link_${'%02d' % (finger_num*4+3)}"/>
             <origin xyz="0 0 ${link2_z}"/>
-            <dynamics damping="10" friction="12"/>
+            <dynamics damping="0.01" friction="0.01"/>
         </joint>
         <!-- [FINGER TIP] -->

Commit message: Create gazebo simulation of the hand

File: src/allegro_hand_description/allegro_hand_description.xacro (robot description, xacro)
@@ -2,4 +2,5 @@
 <robot xmlns:xacro="http://www.ros.org/wiki/xacro" name="allegro_hand">
     <xacro:arg name="chirality" default=""/>
+    <xacro:arg name="gz_plugin_namespace" default=""/>
     <!-- ======================== CHIRALITY PARAMS ========================= -->
     <xacro:property name="suffix" value="$(arg chirality)"/>
@@ -447,4 +448,44 @@
             finger_angle_y="${minus_right * 90*DEG2RAD}"
             />
-    <!-- ============================================================================= -->
+    <!-- ============================= GAZEBO SIMULATION ============================= -->
+    <link name="world"/>
+    <joint name="root_joint" type="fixed">
+                <parent link="world"/>
+                <child link="palm_link"/>
+                <origin rpy="0 0 0" xyz="0 0 0.15"/>
+    </joint>
+    <xacro:macro name="make_transmission" params="joint_num">
+        <transmission name="joint_${'%02d' % joint_num}_trans">
+        <type>transmission_interface/SimpleTransmission</type>
+        <joint name="joint_${'%02d' % joint_num}">
+            <hardwareInterface>hardware_interface/EffortJointInterface</hardwareInterface>
+        </joint>
+        <actuator name="joint_${'%02d' % joint_num}_motor">
+            <mechanicalReduction>1</mechanicalReduction>
+            <hardwareInterface>hardware_interface/EffortJointInterface</hardwareInterface>
+        </actuator>
+        </transmission>
+    </xacro:macro>
+    <xacro:make_transmission joint_num="00"/>
+    <xacro:make_transmission joint_num="01"/>
+    <xacro:make_transmission joint_num="02"/>
+    <xacro:make_transmission joint_num="03"/>
+    <xacro:make_transmission joint_num="04"/>
+    <xacro:make_transmission joint_num="05"/>
+    <xacro:make_transmission joint_num="06"/>
+    <xacro:make_transmission joint_num="07"/>
+    <xacro:make_transmission joint_num="08"/>
+    <xacro:make_transmission joint_num="09"/>
+    <xacro:make_transmission joint_num="10"/>
+    <xacro:make_transmission joint_num="11"/>
+    <xacro:make_transmission joint_num="12"/>
+    <xacro:make_transmission joint_num="13"/>
+    <xacro:make_transmission joint_num="14"/>
+    <xacro:make_transmission joint_num="15"/>
+    <gazebo>
+      <plugin name="ros_control" filename="libgazebo_ros_control.so">
+        <robotNamespace>/$(arg gz_plugin_namespace)</robotNamespace>
+        <legacyModeNS>true</legacyModeNS>
+      </plugin>
+    </gazebo>
 </robot>

Commit message: Slightly increase damping in simulation for stability purposes

File: src/allegro_hand_description/allegro_hand_description.xacro (robot description, xacro)
@@ -119,5 +119,5 @@
             <origin rpy="${finger_angle_r} ${finger_angle_p} ${finger_angle_y}"
                     xyz="${offset_origin_x} ${offset_origin_y} ${offset_origin_z}"/>
-            <dynamics damping="0.01" friction="0.01"/>
+            <dynamics damping="0.1" friction="0.01"/>
         </joint>
         <!-- [LINK 13] -->
@@ -153,5 +153,5 @@
             <child link="link_${'%02d' % (finger_num*4+1)}"/>
             <origin xyz="-0.027 ${minus_left * 0.005} 0.0399"/>
-            <dynamics damping="0.01" friction="0.01"/>
+            <dynamics damping="0.1" friction="0.01"/>
         </joint>
         <!-- [LINK 14] -->
@@ -185,5 +185,5 @@
             <child link="link_${'%02d' % (finger_num*4+2)}"/>
             <origin xyz="0 0 ${link1_t_z}"/>
-            <dynamics damping="0.01" friction="0.01"/>
+            <dynamics damping="0.1" friction="0.01"/>
         </joint>
         <!-- [LINK 15] -->
@@ -218,5 +218,5 @@
             <child link="link_${'%02d' % (finger_num*4+3)}"/>
             <origin xyz="0 0 ${link2_t_z}"/>
-            <dynamics damping="0.01" friction="0.01"/>
+            <dynamics damping="0.1" friction="0.01"/>
         </joint>
         <!-- [FINGER TIP] -->
@@ -285,5 +285,5 @@
             <origin rpy="${finger_angle_r} 0 0"
                     xyz="${offset_origin_x} ${offset_origin_y} ${offset_origin_z}"/>
-            <dynamics damping="0.01" friction="0.01"/>
+            <dynamics damping="0.1" friction="0.01"/>
         </joint>
         <!-- [LINK 1, 5, 9] -->
@@ -317,5 +317,5 @@
             <child link="link_${'%02d' % (finger_num*4+1)}"/>
             <origin xyz="0 0 ${link0_z}"/>
-            <dynamics damping="0.01" friction="0.01"/>
+            <dynamics damping="0.1" friction="0.01"/>
         </joint>
         <!-- [LINK 2, 6, 10]-->
@@ -349,5 +349,5 @@
             <child link="link_${'%02d' % (finger_num*4+2)}"/>
             <origin xyz="0 0 ${link1_z}"/>
-            <dynamics damping="0.01" friction="0.01"/>
+            <dynamics damping="0.1" friction="0.01"/>
         </joint>
         <!-- [LINK 3, 7, 11] -->
@@ -381,5 +381,5 @@
             <child link="link_${'%02d' % (finger_num*4+3)}"/>
             <origin xyz="0 0 ${link2_z}"/>
-            <dynamics damping="0.01" friction="0.01"/>
+            <dynamics damping="0.1" friction="0.01"/>
         </joint>
         <!-- [FINGER TIP] -->
