Commit message: Fix typo : srdf group now indexed by prefix

File: src/allegro_hand_description/allegro_hand_description.srdf.xacro (robot description, xacro)
@@ -38,20 +38,20 @@
         </group>
         <group_state name="open" group="${group_name}">
-            <joint name="left_gripper_joint_00" value="0.0"/>
-            <joint name="left_gripper_joint_01" value="0.0"/>
-            <joint name="left_gripper_joint_02" value="0.0"/>
-            <joint name="left_gripper_joint_03" value="0.0"/>
-            <joint name="left_gripper_joint_04" value="0.0"/>
-            <joint name="left_gripper_joint_05" value="0.0"/>
-            <joint name="left_gripper_joint_06" value="0.0"/>
-            <joint name="left_gripper_joint_07" value="0.0"/>
-            <joint name="left_gripper_joint_08" value="0.0"/>
-            <joint name="left_gripper_joint_09" value="0.0"/>
-            <joint name="left_gripper_joint_10" value="0.0"/>
-            <joint name="left_gripper_joint_11" value="0.0"/>
-            <joint name="left_gripper_joint_12" value="0.4"/>
-            <joint name="left_gripper_joint_13" value="0.0"/>
-            <joint name="left_gripper_joint_14" value="0.0"/>
-            <joint name="left_gripper_joint_15" value="0.0"/>
+            <joint name="${prefix}_joint_00" value="0.0"/>
+            <joint name="${prefix}_joint_01" value="0.0"/>
+            <joint name="${prefix}_joint_02" value="0.0"/>
+            <joint name="${prefix}_joint_03" value="0.0"/>
+            <joint name="${prefix}_joint_04" value="0.0"/>
+            <joint name="${prefix}_joint_05" value="0.0"/>
+            <joint name="${prefix}_joint_06" value="0.0"/>
+            <joint name="${prefix}_joint_07" value="0.0"/>
+            <joint name="${prefix}_joint_08" value="0.0"/>
+            <joint name="${prefix}_joint_09" value="0.0"/>
+            <joint name="${prefix}_joint_10" value="0.0"/>
+            <joint name="${prefix}_joint_11" value="0.0"/>
+            <joint name="${prefix}_joint_12" value="0.4"/>
+            <joint name="${prefix}_joint_13" value="0.0"/>
+            <joint name="${prefix}_joint_14" value="0.0"/>
+            <joint name="${prefix}_joint_15" value="0.0"/>
         </group_state>
     </xacro:macro>
