Commit message: No offset pos in z for standalone urdf

File: allegro_hand/urdf/allegro_hand_on_stand.urdf.xacro (robot description, xacro)
@@ -9,5 +9,5 @@
   <link name="world"/>
   <xacro:allegro_hand chirality="$(arg chirality)" parent="world" prefix="$(arg prefix)">
-    <origin xyz="0.0 0.0 0.25" rpy="0.0 0 0.0"/>
+    <origin xyz="0.0 0.0 0" rpy="0.0 0 0.0"/>
   </xacro:allegro_hand>
 </robot>
