Commit message: Re arrange mesh files

File: allegro_hand_description/allegro_hand_description.urdf.xacro (robot description, xacro)
@@ -1,5 +1,5 @@
 <?xml version="1.0"?>
 <robot xmlns:xacro="http://www.ros.org/wiki/xacro" name="allegro_hand">
-    <xacro:macro name="allegro_hand" params="chirality parent *origin prefix last_links_inertia_factor=1.0">
+    <xacro:macro name="allegro_hand" params="chirality parent *origin prefix ur5_attachment:=false desk_stand:=false last_links_inertia_factor=1.0">
     <!-- ======================== CHIRALITY PARAMS ========================= -->
     <xacro:property name="suffix" value="${chirality}"/>
@@ -59,5 +59,5 @@
         <visual>
             <geometry>
-                <mesh filename="package://allegro_hand_description/meshes/base_link_${suffix}.STL"/>
+                <mesh filename="package://allegro_hand_description/meshes/hand_visuals/base_link_${suffix}.stl"/>
             </geometry>
             <origin rpy="0 0 0" xyz="0 0 0 "/>
@@ -88,5 +88,5 @@
             <visual>
                 <geometry>
-                    <mesh filename="package://allegro_hand_description/meshes/link_12.0_${suffix}.STL"/>
+                    <mesh filename="package://allegro_hand_description/meshes/hand_visuals/link_12_${suffix}.stl"/>
                 </geometry>
                 <material name="black">
@@ -124,5 +124,5 @@
             <visual>
                 <geometry>
-                    <mesh filename="package://allegro_hand_description/meshes/link_13.0.STL"/>
+                    <mesh filename="package://allegro_hand_description/meshes/hand_visuals/link_13.stl"/>
                 </geometry>
                 <material name="black">
@@ -158,5 +158,5 @@
             <visual>
                 <geometry>
-                    <mesh filename="package://allegro_hand_description/meshes/link_14.0.STL"/>
+                    <mesh filename="package://allegro_hand_description/meshes/hand_visuals/link_14.stl"/>
                 </geometry>
                 <material name="black">
@@ -190,5 +190,5 @@
             <visual>
                 <geometry>
-                    <mesh filename="package://allegro_hand_description/meshes/link_15.0.STL"/>
+                    <mesh filename="package://allegro_hand_description/meshes/hand_visuals/link_15.stl"/>
                 </geometry>
                 <material name="black">
@@ -223,5 +223,5 @@
             <visual>
                 <geometry>
-                    <mesh filename="package://allegro_hand_description/meshes/link_15.0_tip.STL"/>
+                    <mesh filename="package://allegro_hand_description/meshes/hand_visuals/link_15_tip.stl"/>
                 </geometry>
                 <material name="white">
@@ -257,5 +257,5 @@
             <visual>
                 <geometry>
-                    <mesh filename="package://allegro_hand_description/meshes/link_0.0.STL"/>
+                    <mesh filename="package://allegro_hand_description/meshes/hand_visuals/link_0.stl"/>
                 </geometry>
                 <material name="black"/>
@@ -290,5 +290,5 @@
             <visual>
                 <geometry>
-                    <mesh filename="package://allegro_hand_description/meshes/link_1.0.STL"/>
+                    <mesh filename="package://allegro_hand_description/meshes/hand_visuals/link_1.stl"/>
                 </geometry>
                 <material name="black"/>
@@ -322,5 +322,5 @@
             <visual>
                 <geometry>
-                    <mesh filename="package://allegro_hand_description/meshes/link_2.0.STL"/>
+                    <mesh filename="package://allegro_hand_description/meshes/hand_visuals/link_2.stl"/>
                 </geometry>
                 <material name="black"/>
@@ -354,5 +354,5 @@
             <visual>
                 <geometry>
-                    <mesh filename="package://allegro_hand_description/meshes/link_3.0.STL"/>
+                    <mesh filename="package://allegro_hand_description/meshes/hand_visuals/link_3.stl"/>
                 </geometry>
                 <material name="black"/>
@@ -386,5 +386,5 @@
             <visual>
                 <geometry>
-                    <mesh filename="package://allegro_hand_description/meshes/link_3.0_tip.STL"/>
+                    <mesh filename="package://allegro_hand_description/meshes/hand_visuals/link_3_tip.stl"/>
                 </geometry>
                 <material name="white">

Commit message: Add xacro args and UR5 fixture

File: allegro_hand_description/allegro_hand_description.urdf.xacro (robot description, xacro)
@@ -14,4 +14,5 @@
     <!-- ======================== BASE PARAMS ========================= -->
     <xacro:property name="palm_link_z" value="0.095"/>
+    <xacro:property name="palm_link_x" value="-0.009300"/>
     <!-- ======================== FINGER PARAMS ======================== -->
     <xacro:property name="links_x" value="0.0196"/>
@@ -54,5 +55,5 @@
     <xacro:property name="limit_3_t_up" value="1.819"/>
     <xacro:property name="limit_3_t_low" value="-0.262"/>
-    <!-- ============================================================================= -->
+    <!-- ============================= HAND and FINGERS ============================== -->
     <!-- PALM -->
     <link name="${prefix}_palm_link">
@@ -67,5 +68,5 @@
         </visual>
         <collision>
-            <origin rpy="0 0 0" xyz="-0.009300 0 -${palm_link_z/2}"/>
+            <origin rpy="0 0 0" xyz="${palm_link_x} 0 -${palm_link_z/2}"/>
             <geometry>
                 <box size="0.0408 0.1130 ${palm_link_z}"/>
@@ -447,10 +448,43 @@
             finger_angle_y="${minus_right * 90*DEG2RAD}"
             />
+    <!-- ================================== SUPPORT ================================== -->
+    <xacro:if value="${ur5_attachment}">
+        <link name="${prefix}_ur5_attachment">
+            <visual>
+                <geometry>
+                    <mesh filename="package://allegro_hand_description/meshes/support_visuals/UR5_attachment.stl" scale="0.001 0.001 0.001"/>
+                </geometry>
+                <material name="grey">
+                    <color rgba=".7 .7 .7 1"/>
+                </material>
+            </visual>
+            <collision>
+                <geometry>
+                    <mesh filename="package://allegro_hand_description/meshes/support_visuals/UR5_attachment_bottom_collision.stl" scale="0.001 0.001 0.001"/>
+                </geometry>
+                <geometry>
+                    <mesh filename="package://allegro_hand_description/meshes/support_visuals/UR5_attachment_top_collision.stl" scale="0.001 0.001 0.001"/>
+                </geometry>
+            </collision>
+            <inertial>
+                <mass value="0.200" />
+                <origin xyz="0 -2.4e-04 1.5e-02" rpy="0 0 0"/>
+                <inertia ixx="1.0e-04" ixy="0"        ixz="0"
+                                       iyy="1.0e-04"  iyz="-4.0e-07"
+                                                      izz="1.2e-04" />
+            </inertial>
+        </link>
+        <joint name="${prefix}_ur5_attachment_joint" type="fixed">
+            <parent link="${prefix}_ur5_attachment"/>
+            <child link="${prefix}_palm_link"/>
+            <origin rpy="0 0 ${90*deg2rad}" xyz="0 ${-palm_link_x} ${0.05+palm_link_z}"/>
+        </joint>
+        <joint name="${prefix}_palm_joint" type="fixed">
+                    <parent link="${parent}"/>
+                    <child link="${prefix}_ur5_attachment"/>
+                    <xacro:insert_block name="origin"/>
+        </joint>
+    </xacro:if>
     <!-- ============================= GAZEBO SIMULATION ============================= -->
-    <joint name="${prefix}_palm_joint" type="fixed">
-                <parent link="${parent}"/>
-                <child link="${prefix}_palm_link"/>
-                <xacro:insert_block name="origin"/>
-    </joint>
     <xacro:macro name="make_transmission" params="joint_num">
         <transmission name="${prefix}_joint_${'%02d' % joint_num}_trans">

Commit message: Move mesh files

File: allegro_hand_description/allegro_hand_description.urdf.xacro (robot description, xacro)
@@ -60,5 +60,5 @@
         <visual>
             <geometry>
-                <mesh filename="package://allegro_hand_description/meshes/hand_visuals/base_link_${suffix}.stl"/>
+                <mesh filename="package://allegro_hand_description/meshes/hand/base_link_${suffix}.stl"/>
             </geometry>
             <origin rpy="0 0 0" xyz="0 0 0 "/>
@@ -89,5 +89,5 @@
             <visual>
                 <geometry>
-                    <mesh filename="package://allegro_hand_description/meshes/hand_visuals/link_12_${suffix}.stl"/>
+                    <mesh filename="package://allegro_hand_description/meshes/hand/link_12_${suffix}.stl"/>
                 </geometry>
                 <material name="black">
@@ -125,5 +125,5 @@
             <visual>
                 <geometry>
-                    <mesh filename="package://allegro_hand_description/meshes/hand_visuals/link_13.stl"/>
+                    <mesh filename="package://allegro_hand_description/meshes/hand/link_13.stl"/>
                 </geometry>
                 <material name="black">
@@ -159,5 +159,5 @@
             <visual>
                 <geometry>
-                    <mesh filename="package://allegro_hand_description/meshes/hand_visuals/link_14.stl"/>
+                    <mesh filename="package://allegro_hand_description/meshes/hand/link_14.stl"/>
                 </geometry>
                 <material name="black">
@@ -191,5 +191,5 @@
             <visual>
                 <geometry>
-                    <mesh filename="package://allegro_hand_description/meshes/hand_visuals/link_15.stl"/>
+                    <mesh filename="package://allegro_hand_description/meshes/hand/link_15.stl"/>
                 </geometry>
                 <material name="black">
@@ -224,5 +224,5 @@
             <visual>
                 <geometry>
-                    <mesh filename="package://allegro_hand_description/meshes/hand_visuals/link_15_tip.stl"/>
+                    <mesh filename="package://allegro_hand_description/meshes/hand/link_15_tip.stl"/>
                 </geometry>
                 <material name="white">
@@ -258,5 +258,5 @@
             <visual>
                 <geometry>
-                    <mesh filename="package://allegro_hand_description/meshes/hand_visuals/link_0.stl"/>
+                    <mesh filename="package://allegro_hand_description/meshes/hand/link_0.stl"/>
                 </geometry>
                 <material name="black"/>
@@ -291,5 +291,5 @@
             <visual>
                 <geometry>
-                    <mesh filename="package://allegro_hand_description/meshes/hand_visuals/link_1.stl"/>
+                    <mesh filename="package://allegro_hand_description/meshes/hand/link_1.stl"/>
                 </geometry>
                 <material name="black"/>
@@ -323,5 +323,5 @@
             <visual>
                 <geometry>
-                    <mesh filename="package://allegro_hand_description/meshes/hand_visuals/link_2.stl"/>
+                    <mesh filename="package://allegro_hand_description/meshes/hand/link_2.stl"/>
                 </geometry>
                 <material name="black"/>
@@ -355,5 +355,5 @@
             <visual>
                 <geometry>
-                    <mesh filename="package://allegro_hand_description/meshes/hand_visuals/link_3.stl"/>
+                    <mesh filename="package://allegro_hand_description/meshes/hand/link_3.stl"/>
                 </geometry>
                 <material name="black"/>
@@ -387,5 +387,5 @@
             <visual>
                 <geometry>
-                    <mesh filename="package://allegro_hand_description/meshes/hand_visuals/link_3_tip.stl"/>
+                    <mesh filename="package://allegro_hand_description/meshes/hand/link_3_tip.stl"/>
                 </geometry>
                 <material name="white">
@@ -453,5 +453,5 @@
             <visual>
                 <geometry>
-                    <mesh filename="package://allegro_hand_description/meshes/support_visuals/UR5_attachment.stl" scale="0.001 0.001 0.001"/>
+                    <mesh filename="package://allegro_hand_description/meshes/support/UR5_attachment.stl" scale="0.001 0.001 0.001"/>
                 </geometry>
                 <material name="grey">
@@ -461,8 +461,8 @@
             <collision>
                 <geometry>
-                    <mesh filename="package://allegro_hand_description/meshes/support_visuals/UR5_attachment_bottom_collision.stl" scale="0.001 0.001 0.001"/>
-                </geometry>
-                <geometry>
-                    <mesh filename="package://allegro_hand_description/meshes/support_visuals/UR5_attachment_top_collision.stl" scale="0.001 0.001 0.001"/>
+                    <mesh filename="package://allegro_hand_description/meshes/support/UR5_attachment_bottom_collision.stl" scale="0.001 0.001 0.001"/>
+                </geometry>
+                <geometry>
+                    <mesh filename="package://allegro_hand_description/meshes/support/UR5_attachment_top_collision.stl" scale="0.001 0.001 0.001"/>
                 </geometry>
             </collision>

Commit message: Add base_screws link and proper stand managment

File: allegro_hand_description/allegro_hand_description.urdf.xacro (robot description, xacro)
@@ -448,5 +448,6 @@
             finger_angle_y="${minus_right * 90*DEG2RAD}"
             />
-    <!-- ================================== SUPPORT ================================== -->
+    <!-- ================================== SUPPORTS ================================== -->
+    <link name="${prefix}_base_screws"/>
     <xacro:if value="${ur5_attachment}">
         <link name="${prefix}_ur5_attachment">
@@ -475,15 +476,80 @@
             </inertial>
         </link>
-        <joint name="${prefix}_ur5_attachment_joint" type="fixed">
-            <parent link="${prefix}_ur5_attachment"/>
-            <child link="${prefix}_palm_link"/>
-            <origin rpy="0 0 ${90*deg2rad}" xyz="0 ${-palm_link_x} ${0.05+palm_link_z}"/>
-        </joint>
-        <joint name="${prefix}_palm_joint" type="fixed">
-                    <parent link="${parent}"/>
-                    <child link="${prefix}_ur5_attachment"/>
-                    <xacro:insert_block name="origin"/>
-        </joint>
     </xacro:if>
+    <xacro:if value="${desk_stand}">
+        <link name="${prefix}_desk_stand">
+            <visual>
+                <material name="grey">
+                    <color rgba=".7 .7 .7 1"/>
+                </material>
+            </visual>
+            <collision>
+                <geometry>
+                    <mesh filename="package://allegro_hand_description/meshes/support/UR5_attachment_bottom_collision.stl" scale="0.001 0.001 0.001"/>
+                </geometry>
+                <geometry>
+                    <mesh filename="package://allegro_hand_description/meshes/support/UR5_attachment_top_collision.stl" scale="0.001 0.001 0.001"/>
+                </geometry>
+            </collision>
+            <inertial>
+                <mass value="0.200" />
+                <origin xyz="0 -2.4e-04 1.5e-02" rpy="0 0 0"/>
+                <inertia ixx="1.0e-04" ixy="0"        ixz="0"
+                                       iyy="1.0e-04"  iyz="-4.0e-07"
+                                                      izz="1.2e-04" />
+            </inertial>
+        </link>
+    </xacro:if>
+<!-- ================================== ORIGIN ================================== -->
+    <joint name="${prefix}_base_screws_joint" type="fixed">
+        <parent link="${prefix}_base_screws"/>
+        <child link="${prefix}_palm_link"/>
+        <origin rpy="0 0 ${90*DEG2RAD}" xyz="0 ${-palm_link_x} ${palm_link_z}"/>
+    </joint>
+    <!-- Desk stand -->
+    <xacro:if value="${desk_stand}">
+        <joint name="${prefix}_parent_joint" type="fixed">
+            <parent link="${parent}"/>
+            <child link="${prefix}_desk_stand"/>
+            <xacro:insert_block name="origin"/>
+        </joint>
+        <joint name="${prefix}_desk_stand_joint" type="fixed">
+            <parent link="${prefix}_desk_stand"/>
+            <child link="${prefix}_base_screws"/>
+            <origin rpy="0 0 0" xyz="0 0 0"/>
+        </joint>
+        <!-- And ur5 attachment -->
+        <xacro:if value="${ur5_attachment}">
+            <joint name="${prefix}_ur5_attachment" type="fixed">
+                <parent link="${prefix}_base_screws"/>
+                <child link="${prefix}_ur5_attachment"/>
+                <origin rpy="0 0 0" xyz="0 0 -0.05"/>
+            </joint>
+        </xacro:if>
+    </xacro:if>
+    <!-- No desk stand -->
+    <xacro:unless value="${desk_stand}">
+        <!-- But UR5 attachmet -->
+        <xacro:if value="${ur5_attachment}">
+            <joint name="${prefix}_ur5_attachment_joint" type="fixed">
+                <parent link="${prefix}_ur5_attachment"/>
+                <child link="${prefix}_base_screws"/>
+                <origin rpy="0 0 0" xyz="0 0 0.05"/>
+            </joint>
+            <joint name="${prefix}_parent_joint" type="fixed">
+                <parent link="${parent}"/>
+                <child link="${prefix}_ur5_attachment"/>
+                <xacro:insert_block name="origin"/>
+            </joint>
+        </xacro:if>
+        <!-- Nothing -->
+        <xacro:unless value="${ur5_attachment}">
+            <joint name="${prefix}_parent_joint" type="fixed">
+                <parent link="${parent}"/>
+                <child link="${prefix}_base_screws"/>
+                <xacro:insert_block name="origin"/>
+            </joint>
+        </xacro:unless>
+    </xacro:unless>
     <!-- ============================= GAZEBO SIMULATION ============================= -->
     <xacro:macro name="make_transmission" params="joint_num">

Commit message: Propper meshes for deskstand

File: allegro_hand_description/allegro_hand_description.urdf.xacro (robot description, xacro)
@@ -480,14 +480,17 @@
         <link name="${prefix}_desk_stand">
             <visual>
+                <geometry>
+                    <mesh filename="package://allegro_hand_description/meshes/support/Allegro_deskstand.stl" scale="0.001 0.001 0.001"/>
+                </geometry>
                 <material name="grey">
-                    <color rgba=".7 .7 .7 1"/>
-                </material>
-            </visual>
-            <collision>
-                <geometry>
-                    <mesh filename="package://allegro_hand_description/meshes/support/UR5_attachment_bottom_collision.stl" scale="0.001 0.001 0.001"/>
-                </geometry>
-                <geometry>
-                    <mesh filename="package://allegro_hand_description/meshes/support/UR5_attachment_top_collision.stl" scale="0.001 0.001 0.001"/>
+                    <color rgba=".8 .8 .8 1"/>
+                </material>
+            </visual>
+            <collision>
+                <geometry>
+                    <mesh filename="package://allegro_hand_description/meshes/support/Allegro_deskstand_bottom_collision.stl" scale="0.001 0.001 0.001"/>
+                </geometry>
+                <geometry>
+                    <mesh filename="package://allegro_hand_description/meshes/support/Allegro_deskstand_top_collision.stl" scale="0.001 0.001 0.001"/>
                 </geometry>
             </collision>
@@ -517,5 +520,5 @@
             <parent link="${prefix}_desk_stand"/>
             <child link="${prefix}_base_screws"/>
-            <origin rpy="0 0 0" xyz="0 0 0"/>
+            <origin rpy="0 0 0" xyz="0 0 0.119"/>
         </joint>
         <!-- And ur5 attachment -->

Commit message: Propper inertia with usage of script

File: allegro_hand_description/allegro_hand_description.urdf.xacro (robot description, xacro)
@@ -469,9 +469,7 @@
             </collision>
             <inertial>
-                <mass value="0.200" />
-                <origin xyz="0 -2.4e-04 1.5e-02" rpy="0 0 0"/>
-                <inertia ixx="1.0e-04" ixy="0"        ixz="0"
-                                       iyy="1.0e-04"  iyz="-4.0e-07"
-                                                      izz="1.2e-04" />
+                <mass value="0.2"/>
+                <origin xyz="0.000 -0.000 0.015" rpy="0  0  0"/>
+                <inertia ixx="1.01e-04" ixy="-1.20e-13" ixz="3.53e-13" iyy="1.04e-04" iyz="-4.03e-07" izz="1.17e-04"/>
             </inertial>
         </link>
@@ -495,11 +493,9 @@
                 </geometry>
             </collision>
-            <inertial>
-                <mass value="0.200" />
-                <origin xyz="0 -2.4e-04 1.5e-02" rpy="0 0 0"/>
-                <inertia ixx="1.0e-04" ixy="0"        ixz="0"
-                                       iyy="1.0e-04"  iyz="-4.0e-07"
-                                                      izz="1.2e-04" />
-            </inertial>
+        <inertial>
+            <mass value="0.3"/>
+            <origin xyz="0.000 0.000 0.018" rpy="0  0  0"/>
+            <inertia ixx="7.09e-04" ixy="-1.32e-14" ixz="1.06e-13" iyy="7.09e-04" iyz="6.26e-15" izz="8.20e-04"/>
+        </inertial>
         </link>
     </xacro:if>

Commit message: Fix minor color error

File: allegro_hand_description/allegro_hand_description.urdf.xacro (robot description, xacro)
@@ -456,6 +456,6 @@
                     <mesh filename="package://allegro_hand_description/meshes/support/UR5_attachment.stl" scale="0.001 0.001 0.001"/>
                 </geometry>
-                <material name="grey">
-                    <color rgba=".7 .7 .7 1"/>
+                <material name="darker_grey">
+                    <color rgba="0.7 0.7 0.7 1"/>
                 </material>
             </visual>
@@ -481,6 +481,6 @@
                     <mesh filename="package://allegro_hand_description/meshes/support/Allegro_deskstand.stl" scale="0.001 0.001 0.001"/>
                 </geometry>
-                <material name="grey">
-                    <color rgba=".8 .8 .8 1"/>
+                <material name="lighter_grey">
+                    <color rgba="0.8 0.8 0.8 1"/>
                 </material>
             </visual>
