Commit message: Fix collision geometries split in two part

File: allegro_hand_description/allegro_hand_description.urdf.xacro (robot description, xacro)
@@ -464,4 +464,6 @@
                     <mesh filename="package://allegro_hand_description/meshes/support/UR5_attachment_bottom_collision.stl" scale="0.001 0.001 0.001"/>
                 </geometry>
+            </collision>
+            <collision>
                 <geometry>
                     <mesh filename="package://allegro_hand_description/meshes/support/UR5_attachment_top_collision.stl" scale="0.001 0.001 0.001"/>
@@ -489,4 +491,6 @@
                     <mesh filename="package://allegro_hand_description/meshes/support/Allegro_deskstand_bottom_collision.stl" scale="0.001 0.001 0.001"/>
                 </geometry>
+            </collision>
+            <collision>
                 <geometry>
                     <mesh filename="package://allegro_hand_description/meshes/support/Allegro_deskstand_top_collision.stl" scale="0.001 0.001 0.001"/>

Commit message: Use convex hull of visual for collision instead of hand made collision boxes

File: allegro_hand_description/allegro_hand_description.urdf.xacro (robot description, xacro)
@@ -62,5 +62,4 @@
                 <mesh filename="package://allegro_hand_description/meshes/hand/base_link_${suffix}.stl"/>
             </geometry>
-            <origin rpy="0 0 0" xyz="0 0 0 "/>
             <material name="black">
                 <color rgba="0.2 0.2 0.2 1"/>
@@ -68,7 +67,6 @@
         </visual>
         <collision>
-            <origin rpy="0 0 0" xyz="${palm_link_x} 0 -${palm_link_z/2}"/>
             <geometry>
-                <box size="0.0408 0.1130 ${palm_link_z}"/>
+                <mesh filename="package://allegro_hand_description/meshes/hand/base_link_${suffix}_collision.stl"/>
             </geometry>
         </collision>
@@ -98,7 +96,7 @@
             <collision>
                 <geometry>
-                    <box size="${link0_t_x} ${link0_t_y} ${link0_t_z}"/>
-                </geometry>
-                <origin rpy="0 0 0" xyz="${-0.0358/2+0.0} ${minus_left * 0.018/2} ${.029/2}"/>
+                    <mesh filename="package://allegro_hand_description/meshes/hand/link_12_${suffix}_collision.stl"/>
+                </geometry>
+                <origin rpy="${zero_right * 180*DEG2RAD} 0 0" xyz="0 0 0"/>
             </collision>
             <inertial>
@@ -132,8 +130,7 @@
             </visual>
             <collision>
-                <geometry>
-                    <box size="${links_x} ${links_y} ${link1_t_z}"/>
-                </geometry>
-                <origin rpy="0 0 0" xyz="0 0 ${link1_t_z/2}"/>
+                 <geometry>
+                    <mesh filename="package://allegro_hand_description/meshes/hand/link_13_collision.stl"/>
+                </geometry>
             </collision>
             <inertial>
@@ -166,7 +163,6 @@
             <collision>
                 <geometry>
-                    <box size="${links_x} ${links_y} ${link2_t_z}"/>
-                </geometry>
-                <origin rpy="0 0 0" xyz="0 0 ${link2_t_z/2}"/>
+                    <mesh filename="package://allegro_hand_description/meshes/hand/link_14_collision.stl"/>
+                </geometry>
             </collision>
             <inertial>
@@ -198,7 +194,6 @@
             <collision>
                 <geometry>
-                    <box size="${links_x} ${links_y} ${link3_t_z-fingerTip_r}"/>
-                </geometry>
-                <origin rpy="0 0 0" xyz="0 0 ${(link3_t_z-fingerTip_r)/2}"/>
+                    <mesh filename="package://allegro_hand_description/meshes/hand/link_15_collision.stl"/>
+                </geometry>
             </collision>
             <inertial>
@@ -232,7 +227,6 @@
             <collision>
                 <geometry>
-                    <sphere radius="${fingerTip_r}"/>
-                </geometry>
-                <origin rpy="0 0 0" xyz="0 0 0"/>
+                    <mesh filename="package://allegro_hand_description/meshes/hand/link_15_tip_collision.stl"/>
+                </geometry>
             </collision>
             <inertial>
@@ -264,7 +258,6 @@
             <collision>
                 <geometry>
-                    <box size="${links_x} ${links_y} ${link0_z}"/>
-                </geometry>
-                <origin rpy="0 0 0" xyz="0 0 ${link0_z/2}"/>
+                    <mesh filename="package://allegro_hand_description/meshes/hand/link_0_collision.stl"/>
+                </geometry>
             </collision>
             <inertial>
@@ -297,7 +290,6 @@
             <collision>
                 <geometry>
-                    <box size="${links_x} ${links_y} ${link1_z}"/>
-                </geometry>
-                <origin rpy="0 0 0" xyz="0 0 ${link1_z/2}"/>
+                    <mesh filename="package://allegro_hand_description/meshes/hand/link_1_collision.stl"/>
+                </geometry>
             </collision>
             <inertial>
@@ -329,7 +321,6 @@
             <collision>
                 <geometry>
-                    <box size="${links_x} ${links_y} ${link2_z}"/>
-                </geometry>
-                <origin rpy="0 0 0" xyz="0 0 ${link2_z/2}"/>
+                    <mesh filename="package://allegro_hand_description/meshes/hand/link_2_collision.stl"/>
+                </geometry>
             </collision>
             <inertial>
@@ -361,7 +352,6 @@
             <collision>
                 <geometry>
-                    <box size="${links_x} ${links_y} ${link3_z-fingerTip_r}"/>
-                </geometry>
-                <origin rpy="0 0 0" xyz="0 0 ${(link3_z-fingerTip_r)/2}"/>
+                    <mesh filename="package://allegro_hand_description/meshes/hand/link_3_collision.stl"/>
+                </geometry>
             </collision>
             <inertial>
@@ -395,5 +385,5 @@
             <collision>
                 <geometry>
-                    <sphere radius="${fingerTip_r}"/>
+                    <mesh filename="package://allegro_hand_description/meshes/hand/link_3_tip_collision.stl"/>
                 </geometry>
             </collision>

Commit message: Minor: indent urdf inertia and unify material colors

File: allegro_hand_description/allegro_hand_description.urdf.xacro (robot description, xacro)
@@ -63,5 +63,5 @@
             </geometry>
             <material name="black">
-                <color rgba="0.2 0.2 0.2 1"/>
+                <color rgba=".2 .2 .2 1"/>
             </material>
         </visual>
@@ -72,10 +72,10 @@
         </collision>
         <inertial>
-        <origin xyz="0 0 ${palm_link_z/2}" rpy="0 0 0"/>
-        <mass value="0.4154"/>
-        <inertia
-            ixx="1e-4" ixy="0.0" ixz="0.0"
-            iyy="1e-4" iyz="0.0"
-            izz="1e-4"/>
+            <origin xyz="0 0 ${palm_link_z/2}" rpy="0 0 0"/>
+            <mass value="0.4154"/>
+            <inertia
+                ixx="1e-4" ixy="0.0" ixz="0.0"
+                iyy="1e-4" iyz="0.0"
+                izz="1e-4"/>
         </inertial>
     </link>
@@ -101,9 +101,9 @@
             </collision>
             <inertial>
-            <mass value="0.0176" />
-            <origin xyz="0 0 0" rpy="0 0 0"/>
-            <inertia ixx="1.892e-05" ixy="7.167e-06" ixz="5.355e-06"
-                     iyy="1.430e-05" iyz="6.806e-06"
-                     izz="1.892e-05" />
+                <mass value="0.0176" />
+                <origin xyz="0 0 0" rpy="0 0 0"/>
+                <inertia ixx="1.892e-05" ixy="7.167e-06" ixz="5.355e-06"
+                        iyy="1.430e-05" iyz="6.806e-06"
+                        izz="1.892e-05" />
             </inertial>
         </link>
@@ -135,9 +135,9 @@
             </collision>
             <inertial>
-            <mass value="0.0119" />
-            <origin xyz="0 0 0" rpy="0 0 0"/>
-            <inertia ixx="4.242e-06" ixy="1.032e-06" ixz="1.603e-06"
-                     iyy="4.523e-06" iyz="1.448e-06"
-                     izz="4.242e-06" />
+                <mass value="0.0119" />
+                <origin xyz="0 0 0" rpy="0 0 0"/>
+                <inertia ixx="4.242e-06" ixy="1.032e-06" ixz="1.603e-06"
+                        iyy="4.523e-06" iyz="1.448e-06"
+                        izz="4.242e-06" />
             </inertial>
         </link>
@@ -159,4 +159,5 @@
                 </geometry>
                 <material name="black">
+                    <color rgba=".2 .2 .2 1"/>
                 </material>
             </visual>
@@ -167,8 +168,8 @@
             </collision>
             <inertial>
-            <mass value="0.038" />
-            <origin xyz="0 0 0" rpy="0 0 0"/>
-            <inertia ixx="4.304e-05" ixy="9.570e-06" ixz="5.120e-06" iyy="1.444e-05"
-                     iyz="1.342e-05" izz="4.304e-05" />
+                <mass value="0.038" />
+                <origin xyz="0 0 0" rpy="0 0 0"/>
+                <inertia ixx="4.304e-05" ixy="9.570e-06" ixz="5.120e-06" iyy="1.444e-05"
+                        iyz="1.342e-05" izz="4.304e-05" />
             </inertial>
         </link>
@@ -190,4 +191,5 @@
                 </geometry>
                 <material name="black">
+                    <color rgba=".2 .2 .2 1"/>
                 </material>
             </visual>
@@ -198,9 +200,9 @@
             </collision>
             <inertial>
-            <mass value="0.0388" />
-            <origin xyz="0 0 0" rpy="0 0 0"/>
-            <inertia ixx="${last_links_inertia_factor * 3.292e-05}" ixy="${last_links_inertia_factor * 8.042e-06}" ixz="${last_links_inertia_factor * 5.228e-06}"
-                     iyy="${last_links_inertia_factor * 1.474e-05}" iyz="${last_links_inertia_factor * 1.128e-05}"
-                     izz="${last_links_inertia_factor * 3.292e-05}" />
+                <mass value="0.0388" />
+                <origin xyz="0 0 0" rpy="0 0 0"/>
+                <inertia ixx="${last_links_inertia_factor * 3.292e-05}" ixy="${last_links_inertia_factor * 8.042e-06}" ixz="${last_links_inertia_factor * 5.228e-06}"
+                        iyy="${last_links_inertia_factor * 1.474e-05}" iyz="${last_links_inertia_factor * 1.128e-05}"
+                        izz="${last_links_inertia_factor * 3.292e-05}" />
             </inertial>
         </link>
@@ -231,9 +233,9 @@
             </collision>
             <inertial>
-            <mass value="0.0168" />
-            <origin xyz="0 0 0" rpy="0 0 0"/>
-            <inertia ixx="${last_links_inertia_factor * 9.680e-07}" ixy="0.0" ixz="0.0"
-                     iyy="${last_links_inertia_factor * 9.680e-07}" iyz="0.0"
-                     izz="${last_links_inertia_factor * 9.680e-07}" />
+                <mass value="0.0168" />
+                <origin xyz="0 0 0" rpy="0 0 0"/>
+                <inertia ixx="${last_links_inertia_factor * 9.680e-07}" ixy="0.0" ixz="0.0"
+                        iyy="${last_links_inertia_factor * 9.680e-07}" iyz="0.0"
+                        izz="${last_links_inertia_factor * 9.680e-07}" />
             </inertial>
         </link>
@@ -254,5 +256,7 @@
                     <mesh filename="package://allegro_hand_description/meshes/hand/link_0.stl"/>
                 </geometry>
-                <material name="black"/>
+                <material name="black">
+                    <color rgba=".2 .2 .2 1"/>
+                </material>
             </visual>
             <collision>
@@ -262,9 +266,9 @@
             </collision>
             <inertial>
-            <mass value="0.0119" />
-            <origin xyz="0 0 0" rpy="0 0 0"/>
-            <inertia ixx="1.016e-06" ixy="0.0" ixz="0.0"
-                     iyy="6.476e-07" iyz="0.0"
-                     izz="1.016e-06" />
+                <mass value="0.0119" />
+                <origin xyz="0 0 0" rpy="0 0 0"/>
+                <inertia ixx="1.016e-06" ixy="0.0" ixz="0.0"
+                        iyy="6.476e-07" iyz="0.0"
+                        izz="1.016e-06" />
             </inertial>
         </link>
@@ -286,5 +290,7 @@
                     <mesh filename="package://allegro_hand_description/meshes/hand/link_1.stl"/>
                 </geometry>
-                <material name="black"/>
+                <material name="black">
+                    <color rgba=".2 .2 .2 1"/>
+                </material>
             </visual>
             <collision>
@@ -294,9 +300,9 @@
             </collision>
             <inertial>
-            <mass value="0.065" />
-            <origin xyz="0 0 0" rpy="0 0 0"/>
-            <inertia ixx="7.956e-05" ixy="1.719e-05" ixz="8.758e-06"
-                     iyy="2.470e-05" iyz="2.413e-05"
-                     izz="7.956e-05" />
+                <mass value="0.065" />
+                <origin xyz="0 0 0" rpy="0 0 0"/>
+                <inertia ixx="7.956e-05" ixy="1.719e-05" ixz="8.758e-06"
+                        iyy="2.470e-05" iyz="2.413e-05"
+                        izz="7.956e-05" />
             </inertial>
         </link>
@@ -317,5 +323,7 @@
                     <mesh filename="package://allegro_hand_description/meshes/hand/link_2.stl"/>
                 </geometry>
-                <material name="black"/>
+                <material name="black">
+                    <color rgba=".2 .2 .2 1"/>
+                </material>
             </visual>
             <collision>
@@ -325,9 +333,9 @@
             </collision>
             <inertial>
-            <mass value="0.0355" />
-            <origin xyz="0 0 0" rpy="0 0 0"/>
-            <inertia ixx="${last_links_inertia_factor * 2.639e-05}" ixy="${last_links_inertia_factor * 6.679e-06}" ixz="${last_links_inertia_factor * 4.783e-06}"
-                     iyy="${last_links_inertia_factor * 1.349e-05}" iyz="${last_links_inertia_factor * 9.372e-06}"
-                     izz="${last_links_inertia_factor * 2.639e-05}" />
+                <mass value="0.0355" />
+                <origin xyz="0 0 0" rpy="0 0 0"/>
+                <inertia ixx="${last_links_inertia_factor * 2.639e-05}" ixy="${last_links_inertia_factor * 6.679e-06}" ixz="${last_links_inertia_factor * 4.783e-06}"
+                        iyy="${last_links_inertia_factor * 1.349e-05}" iyz="${last_links_inertia_factor * 9.372e-06}"
+                        izz="${last_links_inertia_factor * 2.639e-05}" />
             </inertial>
         </link>
@@ -348,5 +356,7 @@
                     <mesh filename="package://allegro_hand_description/meshes/hand/link_3.stl"/>
                 </geometry>
-                <material name="black"/>
+                <material name="black">
+                    <color rgba=".2 .2 .2 1"/>
+                </material>
             </visual>
             <collision>
@@ -356,9 +366,9 @@
             </collision>
             <inertial>
-            <mass value="0.0096" />
-            <origin xyz="0 0 0" rpy="0 0 0"/>
-            <inertia ixx="${last_links_inertia_factor * 4.701e-06}" ixy="${last_links_inertia_factor * 1.255e-06}" ixz="${last_links_inertia_factor * 1.293e-06}"
-                     iyy="${last_links_inertia_factor * 3.649e-06}" iyz="${last_links_inertia_factor * 1.762e-06}"
-                     izz="${last_links_inertia_factor * 4.701e-06}" />
+                <mass value="0.0096" />
+                <origin xyz="0 0 0" rpy="0 0 0"/>
+                <inertia ixx="${last_links_inertia_factor * 4.701e-06}" ixy="${last_links_inertia_factor * 1.255e-06}" ixz="${last_links_inertia_factor * 1.293e-06}"
+                        iyy="${last_links_inertia_factor * 3.649e-06}" iyz="${last_links_inertia_factor * 1.762e-06}"
+                        izz="${last_links_inertia_factor * 4.701e-06}" />
             </inertial>
         </link>
@@ -390,8 +400,8 @@
             <inertial>
             <mass value="0.0168" />
-            <origin xyz="0 0 0" rpy="0 0 0"/>
-            <inertia ixx="${last_links_inertia_factor * 9.680e-07}" ixy="0.0" ixz="0.0"
-                     iyy="${last_links_inertia_factor * 9.680e-07}" iyz="0.0"
-                     izz="${last_links_inertia_factor * 9.680e-07}" />
+                <origin xyz="0 0 0" rpy="0 0 0"/>
+                <inertia ixx="${last_links_inertia_factor * 9.680e-07}" ixy="0.0" ixz="0.0"
+                        iyy="${last_links_inertia_factor * 9.680e-07}" iyz="0.0"
+                        izz="${last_links_inertia_factor * 9.680e-07}" />
             </inertial>
         </link>

Commit message: Fix velocity limit value in urdf

File: allegro_hand_description/allegro_hand_description.urdf.xacro (robot description, xacro)
@@ -110,5 +110,5 @@
         <joint name="${prefix}_joint_${'%02d' % (finger_num*4+0)}" type="revolute">
             <axis xyz="${minus_right} 0 0"/>
-            <limit effort="0.71" velocity="0.12"
+            <limit effort="0.71" velocity="9.5"
                 lower="${limit_0_t_low+joint_safety_margin}"
                 upper="${limit_0_t_up-joint_safety_margin}"/>
@@ -144,5 +144,5 @@
         <joint name="${prefix}_joint_${'%02d' % (finger_num*4+1)}" type="revolute">
             <axis xyz="0 0 ${minus_left}"/>
-            <limit effort="0.71" velocity="0.12"
+            <limit effort="0.71" velocity="9.5"
                 lower="${limit_1_t_low+joint_safety_margin}"
                 upper="${limit_1_t_up-joint_safety_margin}"/>
@@ -176,5 +176,5 @@
         <joint name="${prefix}_joint_${'%02d' % (finger_num*4+2)}" type="revolute">
             <axis xyz="0 1 0"/>
-            <limit effort="0.71" velocity="0.12"
+            <limit effort="0.71" velocity="9.5"
                 lower="${limit_2_t_low+joint_safety_margin}"
                 upper="${limit_2_t_up-joint_safety_margin}"/>
@@ -209,5 +209,5 @@
         <joint name="${prefix}_joint_${'%02d' % (finger_num*4+3)}" type="revolute">
             <axis xyz="0 1 0"/>
-            <limit effort="0.71" velocity="0.12"
+            <limit effort="0.71" velocity="9.5"
                 lower="${limit_3_t_low+joint_safety_margin}"
                 upper="${limit_3_t_up-joint_safety_margin}"/>
@@ -275,5 +275,5 @@
         <joint name="${prefix}_joint_${'%02d' % (finger_num*4+0)}" type="revolute">
             <axis xyz="0 0 1"/>
-            <limit effort="0.71" velocity="0.12"
+            <limit effort="0.71" velocity="9.5"
                 lower="${limit_0_low+joint_safety_margin}"
                 upper="${limit_0_up-joint_safety_margin}"/>
@@ -308,5 +308,5 @@
         </link>
         <joint name="${prefix}_joint_${'%02d' % (finger_num*4+1)}" type="revolute">
-            <limit effort="0.71" velocity="0.12"
+            <limit effort="0.71" velocity="9.5"
                 lower="${limit_1_low+joint_safety_margin}"
                 upper="${limit_1_up-joint_safety_margin}"/>
@@ -342,5 +342,5 @@
         <joint name="${prefix}_joint_${'%02d' % (finger_num*4+2)}" type="revolute">
             <axis xyz="0 1 0"/>
-            <limit effort="0.71" velocity="0.12"
+            <limit effort="0.71" velocity="9.5"
                 lower="${limit_2_low+joint_safety_margin}"
                 upper="${limit_2_up-joint_safety_margin}"/>
@@ -375,5 +375,5 @@
         <joint name="${prefix}_joint_${'%02d' % (finger_num*4+3)}" type="revolute">
             <axis xyz="0 1 0"/>
-            <limit effort="0.71" velocity="0.12"
+            <limit effort="0.71" velocity="9.5"
                 lower="${limit_3_low+joint_safety_margin}"
                 upper="${limit_3_up-joint_safety_margin}"/>
@@ -586,5 +586,5 @@
     <plugin name="${prefix}_ros_control" filename="libgazebo_ros_control_select_joints.so">
         <robotNamespace>/${prefix}</robotNamespace>
-        <legacyModeNS>true</legacyModeNS>
+        <legacyModeNS>false</legacyModeNS>
         <joints>
             ${prefix}_joint_00
